File: pcb/swmeter.kicad_pcb (KiCad board)
At the start: 2 copper layers, 53 x 66 mm, 29 parts, among them J0 Conn_01x02_Female, J1 AudioPlug, J2 Conn_Coaxial, J3 Conn_01x03_Female, J4 Conn_01x03_Female, SW1 SW_SPDT, SW2 SW_SPDT, SW3 SW_DIP_x03, U1 LM3914N

Commit message: -mounting with gnd -removed orientation crosses
Parts:
- removed REF1: MountingHole_3.2mm_M3_Pad_Via, MountingHole:MountingHole_3.2mm_M3_Pad_Via
- removed REF5, REF55: RoHS-Logo_6mm_SilkScreen, Symbol:RoHS-Logo_6mm_SilkScreen
- added REF77**: ESD-Logo_13.2x12mm_SilkScreen, Symbol:ESD-Logo_13.2x12mm_SilkScreen, B.Cu at (216.3, 94.0)
- added REF8**: KiCad-Logo2_5mm_SilkScreen, Symbol:KiCad-Logo2_5mm_SilkScreen, F.Cu at (213.4, 141.7)
- added REF88**: KiCad-Logo2_5mm_SilkScreen, Symbol:KiCad-Logo2_5mm_SilkScreen, B.Cu at (213.4, 141.6)
- added REF99**: MountingHole_3.2mm_M3_Pad, MountingHole:MountingHole_3.2mm_M3_Pad, F.Cu at (221.8, 123.6)
- moved REF3 27.6 mm to (214.1, 129.4)
- moved REF33 27.5 mm to (214.1, 129.3)
- moved REF00 11.4 mm to (214.0, 122.7), turned to 90 degrees
- moved REF0 11.4 mm to (214.1, 122.8), turned to -90 degrees
- moved G9 7.97 mm to (211.0, 119.0)
- moved G99 7.75 mm to (211.1, 119.1)
- moved G11 1.59 mm to (216.6, 109.4)
- moved G1 1.29 mm to (216.8, 109.5)
- moved G2 1.18 mm to (230.6, 124.2)
- moved G22 1.00 mm to (230.7, 124.8)
- renumbered REF** to REF7**
Connections:
- SW1 pad : (no net) -> GND
- SW2 pad : (no net) -> GND
Routing:
- net Net-(BAR1-Pad1): track 122.4 -> 124.5 mm
Other:
- board text added: "+"
- board text added: "GND"
- board text added: "LED1"
- board text added: "LED_Bargraph"
- board text added: "Mode"
- board text added: "RHi"
- board text added: "RLo"
- board text added: "RefAdj"
- board text added: "RefOut"
- board text added: "RoHS"
- board text added: "VCC"
- board text removed: "LED-Bargraph"
